File: MotorBoardv3_2/ChargeCircuit.kicad_sch (KiCad schematic)
At the start: 14 parts, among them J20 Barrel_Jack, Q1 TIP42A, U7 MAX712CSE

Commit message: Initial Charge Controller layout
Connections:
- net V+: now reaches C12.1, R8.2, U7.15 (V+), U7.5 (THI)
Changed lines of the file:
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@@
+		)
+	)
+	(label "V+"
+		(at 115.57 64.77 0)
+		(fields_autoplaced yes)
+		(effects
+			(font
+				(size 1.27 1.27)
+			)
+			(justify left bottom)
 		)
 	)

Commit message: Label adjustements
Connections:
- net DRV: now reaches C13.2, Q1.1 (B), R11.2, U7.14 (DRV)
- net REF: now reaches R9.1, U7.1 (VLIMIT), U7.16 (REF)
- net TEMP: now reaches R10.1, R9.2, U7.7 (TEMP)
Changed lines of the file:
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@@
+		)
+	)
+	(label "DRV"
+		(at 134.62 49.53 0)
+		(fields_autoplaced yes)
+		(effects
+			(font
+				(size 1.27 1.27)
+			)
+			(justify left bottom)
+		)
+	)
+	(label "TEMP"
+		(at 125.73 78.74 0)
+		(fields_autoplaced yes)
+		(effects
+			(font
+				(size 1.27 1.27)
+			)
+			(justify left bottom)
 		)
 	)
@@
 		(fields_autoplaced yes)
 		(effects
+			(font
+				(size 1.27 1.27)
+			)
+			(justify left bottom)
+		)
+	)
+	(label "REF"
+		(at 123.19 71.12 0)
+		(fields_autoplaced yes)
+		(effects
