File: MotorBoardv3_2/RN4871.kicad_sch (KiCad schematic)
At the start: 2 parts, among them U6 RN4871

Commit message: Completed Schematic w/ charge circuit, voltmeter, bluetooth, Reflective Sensor Port
Parts:
- C10: value 10u -> 10uF; footprint (none) -> RSLK2:C_0603_1608Metric
Changed lines of the file:
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@@
 		(dnp no)
 		(fields_autoplaced yes)
-		(property "Reference" "#PWR021"
+		(property "Reference" "#PWR0101"
 			(at 121.92 50.8 0)
 			(effects
@@
 			(project ""
 				(path "/69b823fd-c065-40ff-9bb9-c5835555f3eb/08191d98-e039-4013-a446-27ee810ce84e"
-					(reference "#PWR021")
+					(reference "#PWR0101")
 					(unit 1)
 				)
@@
 			)
 		)
-		(property "Value" "10u"
+		(property "Value" "10uF"
 			(at 125.73 40.6399 0)
 			(effects
@@
 			)
 		)
-		(property "Footprint" ""
+		(property "Footprint" "RSLK2:C_0603_1608Metric"
 			(at 122.8852 43.18 0)
 			(effects

Commit message: routed RN4871 eval board pins
Also changed the positions of some silkscreen labels
Parts:
- U6: footprint RF_Module:Microchip_RN4871 -> VoltageDisplay:RN4871_eval
Changed lines of the file:
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@@
 			)
 		)
-		(property "Footprint" "RF_Module:Microchip_RN4871"
+		(property "Footprint" "VoltageDisplay:RN4871_eval"
 			(at 107.95 81.28 0)
 			(effects
